Commit message: Improved simple shapes in head for Atlas v4 and v5

File: atlas_description/urdf/atlas_v4_simple_shapes.urdf (robot description, URDF)
Before this commit: robot drc_skeleton, 34 links, 34 joints
Links:
- link utorso: geometry collision box size=0.2 0.25 0.01; collision box size=0.500175 0.35 0.5

File: atlas_description/urdf/atlas_v5_simple_shapes.urdf (robot description, URDF)
Before this commit: robot drc_skeleton, 34 links, 34 joints
Links:
- link utorso: geometry collision box size=0.2 0.25 0.01; collision box size=0.500175 0.35 0.5
